File: schematic/mcupedal.kicad_sch (KiCad schematic)
At the start: 23 parts, among them J1 Barrel_Jack_Switch, J2 AudioJack3_Switch, J3 Screw_Terminal_01x02, J4 AudioJack3_Switch, J5 Screw_Terminal_01x03, J6 Screw_Terminal_01x03, U1 AMS1117-3.3, U2 footswitch, U3 Opamp_Dual, U4 ATtiny85-20P

Commit message: feat(pcb): swap dc pins
Parts:
- added R1: 100, Resistor_SMD:R_1206_3216Metric, symbol Device:R
- U2, U3, U4: Spice_Netlist_Enabled (none) -> N; Spice_Primitive (none) -> R
- renumbered R1 to R2, R2 to R3, R3 to R4, R4 to R5
Connections:
- net +3V3: now also R1.1
- net +9V: now also J1.2; no longer J1.1
- net GND: now also J1.1, R1.2; no longer J1.2
Other:
- moved on the sheet: C1, C2, C3, C4, C5, C6, C7, C8, C9, J1, J2, J3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

Commit message: feat(schematic): cleanup
Parts:
- R3: value 200K -> 220K
Changed lines of the file:
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@@
       (effects (font (size 1.27 1.27)) (justify left))
     )
-    (property "Value" "200K" (id 1) (at 113.03 77.4699 0)
+    (property "Value" "220K" (id 1) (at 113.03 77.4699 0)
       (effects (font (size 1.27 1.27)) (justify left))
     )
@@
     )
     (path "/0203cc9c-33f9-456b-b7e0-9878224d49b4"
-      (reference "R3") (unit 1) (value "200K") (footprint "Resistor_SMD:R_1206_3216Metric")
+      (reference "R3") (unit 1) (value "220K") (footprint "Resistor_SMD:R_1206_3216Metric")
     )
     (path "/15f70aa3-6aa7-4ce9-b7d3-7b19f353c8c4"

Commit message: chore(tidy): removed unused components
Parts:
- removed C6, C9: 100nF, Capacitor_SMD:C_1206_3216Metric, symbol Device:C
- removed J5, J6: Screw_Terminal_01x03, TerminalBlock_Phoenix:TerminalBlock_Phoenix_MPT-0,5-3-2.54_1x03_P2.54mm_Horizontal, symbol Connector:Screw_Terminal_01x03
- removed R1: 100, Resistor_SMD:R_1206_3216Metric, symbol Device:R
- removed U1: AMS1117-3.3, Package_TO_SOT_SMD:SOT-223-3_TabPin2, symbol Regulator_Linear:AMS1117-3.3
- added U1: HT75xx-1-SOT89, Package_TO_SOT_SMD:SOT-89-3, symbol Regulator_Linear:HT75xx-1-SOT89
- renumbered C7 to C6, C8 to C7, R2 to R1, R3 to R2, R4 to R3, R5 to R4
Connections:
- net +3V3: now also U1.3 (VOUT)
- net +9V: now also U1.2 (VIN)
- net GND: now also U1.1 (GND)
- no-connect marks 10 -> 12
